Commit message: Changed lids step files

File: aur_description/urdf/aur.xacro (robot description, xacro)
@@ -2,5 +2,5 @@
 <robot name="aur" xmlns:xacro="http://www.ros.org/wiki/xacro">
 <xacro:include filename="$(find aur_description)/urdf/materials.xacro" />
-<xacro:include filename="$(find aur_description)/urdf/aur.trans"/>
+<!--<xacro:include filename="$(find aur_description)/urdf/aur.trans"/>-->
 <xacro:include filename="$(find aur_description)/gazebo/aur_materials.gazebo" />
 <xacro:include filename="$(find aur_description)/gazebo/aur_physics.gazebo" />
@@ -155,5 +155,5 @@
     <origin rpy="0 0 0" xyz="-0.225 -0.0002 -0.25"/>
     <geometry>
-      <mesh filename="package://aur_description/meshes/lid.stl" scale="0.001 0.001 0.001"/>
+      <mesh filename="package://aur_description/meshes/lid.stl" scale="1.00 1.00 1.00"/>
     </geometry>
     <material name="white"/>
@@ -193,7 +193,7 @@
   </inertial>
   <visual>
-    <origin rpy="0 0 0" xyz="0.035 -0.015 -0.28"/>
-    <geometry>
-      <mesh filename="package://aur_description/meshes/electronics_lid.stl" scale="0.001 0.001 0.001"/>
+    <origin rpy="0 0 0" xyz="0.035 -0.015 -0.266"/>
+    <geometry>
+      <mesh filename="package://aur_description/meshes/electronics_lid.stl" scale="1.00 1.00 1.00"/>
     </geometry>
     <material name="blue"/>
